File: TickiT_WS2812B_PCB/TickiT_WS2812B.kicad_pcb (KiCad board)
At the start: 2 copper layers, 80 x 80 mm, 33 parts, among them J1 Battery, J2 Power, J3 Switch, Q1 FS8205A, U1 ATtiny402-SS, U2 TP4056-42-ESOP8, U3 DW01A

Commit message: PCB V0.1
Parts:
- added C10: 100n, Capacitor_SMD:C_0603_1608Metric_Pad1.08x0.95mm_HandSolder, F.Cu at (179.9, 108.0)
- added C11: 100n, Capacitor_SMD:C_0603_1608Metric_Pad1.08x0.95mm_HandSolder, F.Cu at (171.9, 121.9)
- added C12: 100n, Capacitor_SMD:C_0603_1608Metric_Pad1.08x0.95mm_HandSolder, F.Cu at (158.0, 129.9)
- added C13: 100n, Capacitor_SMD:C_0603_1608Metric_Pad1.08x0.95mm_HandSolder, F.Cu at (142.0, 129.9)
- added C14: 100n, Capacitor_SMD:C_0603_1608Metric_Pad1.08x0.95mm_HandSolder, F.Cu at (128.1, 121.9)
- added C15: 100n, Capacitor_SMD:C_0603_1608Metric_Pad1.08x0.95mm_HandSolder, F.Cu at (120.1, 108.0)
- added C16: 100n, Capacitor_SMD:C_0603_1608Metric_Pad1.08x0.95mm_HandSolder, F.Cu at (120.1, 92.0)
- added C17: 100n, Capacitor_SMD:C_0603_1608Metric_Pad1.08x0.95mm_HandSolder, F.Cu at (128.1, 78.1)
- added C18: 100n, Capacitor_SMD:C_0603_1608Metric_Pad1.08x0.95mm_HandSolder, F.Cu at (142.0, 70.1)
- added C7: 100n, Capacitor_SMD:C_0603_1608Metric_Pad1.08x0.95mm_HandSolder, F.Cu at (158.0, 70.1)
- added C8: 100n, Capacitor_SMD:C_0603_1608Metric_Pad1.08x0.95mm_HandSolder, F.Cu at (171.9, 78.1)
- added C9: 100n, Capacitor_SMD:C_0603_1608Metric_Pad1.08x0.95mm_HandSolder, F.Cu at (179.9, 92.0)
- added H1: MountingHole, MountingHole:MountingHole_3mm, F.Cu at (150.0, 68.0)
- added H2: MountingHole, MountingHole:MountingHole_3mm, F.Cu at (177.7, 116.0)
- added H3: MountingHole, MountingHole:MountingHole_3mm, F.Cu at (122.3, 116.0)
- added R7: 100R, Resistor_SMD:R_0603_1608Metric_Pad0.98x0.95mm_HandSolder, F.Cu at (146.0, 77.0)
- added TP1: G, TestPoint:TestPoint_Pad_D1.0mm, F.Cu at (145.2, 83.6)
- added TP2: +5V, TestPoint:TestPoint_Pad_D1.0mm, F.Cu at (145.2, 86.1)
- added TP3: D, TestPoint:TestPoint_Pad_D1.0mm, F.Cu at (145.2, 81.0)
- added U2: TSOP382xx, OptoDevice:Vishay_MINICAST-3Pin, F.Cu at (160.5, 82.9)
- moved C6 9.81 mm to (174.0, 108.0)
- moved D9 9.15 mm to (183.9, 109.1), turned to -105 degrees
- moved D8 9.15 mm to (174.8, 124.8), turned to -135 degrees
- moved D10 9.15 mm to (183.9, 91.0), turned to -75 degrees
- moved D7 9.14 mm to (159.1, 133.8), turned to -165 degrees
- moved D11 9.14 mm to (174.8, 75.3), turned to -45 degrees
- moved D12 9.14 mm to (159.1, 66.2), turned to -15 degrees
- moved D6 9.14 mm to (141.0, 133.8), turned to 165 degrees
- moved D1 9.13 mm to (141.0, 66.2), turned to 15 degrees
- moved D5 9.13 mm to (125.3, 124.8), turned to 135 degrees
- moved D4 9.13 mm to (116.2, 109.1), turned to 105 degrees
- moved D2 9.13 mm to (125.3, 75.3), turned to 45 degrees
- moved D3 9.12 mm to (116.2, 91.0), turned to 75 degrees
- moved C2 1.75 mm to (152.0, 86.9)
- moved C1 1.49 mm to (152.0, 85.4)
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- renumbered U2 to U4
Connections:
- D1 pad 4: DIN -> Net-(D1-DIN)
- U1 pad 2: unconnected-(U1-PA6-Pad2) -> IR
- U1 pad 4: DIN -> DOUT
- U1 pad 5: SW -> DIN
- U1 pad 6: unconnected-(U1-~{RESET}/PA0-Pad6) -> DATA
- U1 pad 7: DOUT -> SW
Routing:
- net +BATT: track 97.8 -> 182.5 mm
- net DIN: track 24.3 -> 3.45 mm
- net Net-(D1-DIN): track 0.00 -> 14.6 mm
- net DOUT: track 23.2 -> 13.8 mm
- net IR: track 0.00 -> 7.78 mm
- net GND: track 20.9 -> 24.7 mm, vias 4 -> 16
- net DATA: track 0.00 -> 2.80 mm
- net SW: track 16.0 -> 14.8 mm
- net Net-(D10-DIN): track 13.9 -> 14.7 mm
- net Net-(D6-DOUT): track 13.9 -> 13.4 mm
- net Net-(D3-DOUT): track 13.9 -> 13.4 mm
Other:
- board text added: "+"
- board text added: "Tomatito Lamp"
- board text added: "V0.1"
