File: TickiT_WS2812B_PCB/TickiT_WS2812B.kicad_sch (KiCad schematic)
At the start: 17 parts, among them J1 Battery, J2 Power, J3 Switch, U1 ATtiny402-SS, U2 TP4056-42-ESOP8

Commit message: PCB routing
Parts:
- added C1: 1u, Capacitor_SMD:C_0603_1608Metric_Pad1.08x0.95mm_HandSolder, symbol Device:C
- added C2, C4, C5: 100n, Capacitor_SMD:C_0603_1608Metric_Pad1.08x0.95mm_HandSolder, symbol Device:C
- added C3, C6: 10u, Capacitor_SMD:C_0603_1608Metric_Pad1.08x0.95mm_HandSolder, symbol Device:C
- added D13: Blue, LED_SMD:LED_0603_1608Metric_Pad1.05x0.95mm_HandSolder, symbol Device:LED
- added D14: Red, LED_SMD:LED_0603_1608Metric_Pad1.05x0.95mm_HandSolder, symbol Device:LED
- added Q1: FS8205A, SamacSys_Parts:SOP65P640X120-8N, symbol SamacSys_Parts:FS8205A
- added R1, R2, R4: 1k, Resistor_SMD:R_0603_1608Metric_Pad0.98x0.95mm_HandSolder, symbol Device:R
- added R3: R, Resistor_SMD:R_0603_1608Metric_Pad0.98x0.95mm_HandSolder, symbol Device:R
- added R5: 100, Resistor_SMD:R_0603_1608Metric_Pad0.98x0.95mm_HandSolder, symbol Device:R
- added R6: 0R, Resistor_SMD:R_0603_1608Metric_Pad0.98x0.95mm_HandSolder, symbol Device:R
- added U3: DW01A, Package_TO_SOT_SMD:SOT-23-6, symbol Battery_Management:DW01A
- J1, J2, J3: footprint (none) -> SamacSys_Parts:S2BPHSM4TBLFSN
Connections:
- net +5V is gone; now on net +BATT: D1.1 (VDD), D10.1 (VDD), D11.1 (VDD), D12.1 (VDD), D2.1 (VDD), D3.1 (VDD), D4.1 (VDD), D5.1 (VDD), D6.1 (VDD), D7.1 (VDD), D8.1 (VDD), D9.1 (VDD)
- net DIN: now also U1.4 (PA1)
- net DOUT: now also U1.7 (PA3)
- net GND: now also J2.1 (Pin_1), J3.2 (Pin_2), U1.8 (GND), U2.1 (TEMP), U2.3 (GND), U2.9 (EPAD), C1.2, C2.2, C3.2, C4.2, C6.2, Q1.2 (S1_1), Q1.3 (S1_2), R3.1, R4.1, R6.1
- net Vin+: now reaches J2.2 (Pin_2)
- net Vin+: now also U2.4 (V_{CC}), U2.8 (CE), C3.1, C4.1, D13.2 (A), D14.2 (A)
- net +BATT: now reaches U1.1 (VCC)
- net +BATT: now also J1.2 (Pin_2), U2.5 (BAT), C1.1, C2.1, C6.1, R5.2
- net SW: now reaches U1.5 (PA2)
- net SW: now also J3.1 (Pin_1)
- net at U2.2 (PROG): now also R3.2
- net at U2.6 (~{STDBY}): now also R1.1
- net at U2.7 (~{CHRG}): now also R2.1
- net -BATT: now reaches J1.1 (Pin_1)
- net -BATT: now also C5.2, Q1.6 (S2_1), Q1.7 (S2_2), R6.2, U3.6 (GND)
- new net: C5.1, R5.1, U3.5 (VCC)
- new net: D13.1 (K), R1.2
- new net: D14.1 (K), R2.2
- new net: Q1.4 (G1), U3.3 (OC)
- new net: Q1.5 (G2), U3.1 (OD)
- new net: R4.2, U3.2 (CS)
- no-connect marks 0 -> 5
Other:
- company: (none) -> GP
- title: (none) -> TickiT Mood Light WS2812b
- moved on the sheet: J1, J2, J3, U2

Commit message: PCB V0.1
Parts:
- added C10, C11, C12, C13, C14, C15, C16, C17, C18, C7, C8, C9: 100n, Capacitor_SMD:C_0603_1608Metric_Pad1.08x0.95mm_HandSolder, symbol Device:C
- added H1, H2, H3: MountingHole, MountingHole:MountingHole_3mm, symbol Mechanical:MountingHole
- added R7: 100R, Resistor_SMD:R_0603_1608Metric_Pad0.98x0.95mm_HandSolder, symbol Device:R
- added TP1: G, TestPoint:TestPoint_Pad_D1.0mm, symbol Connector:TestPoint
- added TP2: +5V, TestPoint:TestPoint_Pad_D1.0mm, symbol Connector:TestPoint
- added TP3: D, TestPoint:TestPoint_Pad_D1.0mm, symbol Connector:TestPoint
- added U2: TSOP382xx, OptoDevice:Vishay_MINICAST-3Pin, symbol Interface_Optical:TSOP382xx
- renumbered U2 to U4
Connections:
- net +BATT: now also C10.1, C11.1, C12.1, C13.1, C14.1, C15.1, C16.1, C17.1, C18.1, C7.1, C8.1, C9.1, TP2.1, U2.3 (Vs)
- net DIN: now also U1.5 (PA2), R7.1; no longer D1.4 (DIN), U1.4 (PA1)
- net DOUT: now also U1.4 (PA1); no longer U1.7 (PA3)
- net GND: now also C10.2, C11.2, C12.2, C13.2, C14.2, C15.2, C16.2, C17.2, C18.2, C7.2, C8.2, C9.2, TP1.1, U2.2 (GND)
- net SW: now also U1.7 (PA3); no longer U1.5 (PA2)
- net IR: now reaches U1.2 (PA6)
- net IR: now also U2.1 (OUT)
- net DATA: now reaches U1.6 (~{RESET}/PA0)
- net DATA: now also TP3.1
- new net: D1.4 (DIN), R7.2
- no-connect marks 5 -> 3
Other:
- note added: "Prog"
- moved on the sheet: C1, C2, D1, D10, D11, D12, D2, D3, D4, D5, D6, D7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
